File: KiCad_Files/VacuumATM_wCoinDispenser/VacuumATM_wCoinDispenser.kicad_sch (KiCad schematic)
At the start: 10 parts, among them J1 VacButton, J2 Neopixel, J3 9g Servo, J4 User2_Button, J5 User1_Button

Commit message: Updates to KiCAD, images
Parts:
- added J6: ResetButton, TerminalBlock_Phoenix:TerminalBlock_Phoenix_MKDS-1,5-2_1x02_P5.00mm_Horizontal, symbol Connector:Screw_Terminal_01x02
- J1: value VacButton -> CamButton
Connections:
- net GND: now also J6.2 (Pin_2)
- net at A1.1 (~{RESET}): now also J6.1 (Pin_1)
Changed lines of the file:
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@@
+	(wire
+		(pts
+			(xy 160.02 48.26) (xy 154.94 48.26)
+		)
+		(stroke
+			(width 0)
+			(type default)
+		)
+	)
+	(wire
+		(pts
+			(xy 160.02 45.72) (xy 146.05 45.72)
+		)
+		(stroke
+			(width 0)
+			(type default)
+		)
+	)
 	(wire
 		(pts
@@
 		)
 	)
+	(wire
+		(pts
+			(xy 146.05 45.72) (xy 146.05 53.34)
+		)
+		(stroke
+			(width 0)
+			(type default)
+		)
+	)
+	(wire
+		(pts
+			(xy 154.94 48.26) (xy 154.94 50.8)
+		)
+		(stroke
+			(width 0)
+			(type default)
+		)
+	)
 	(symbol
 		(lib_id "Connector:Screw_Terminal_01x02")
@@
 			)
 		)
-		(property "Value" "VacButton"
+		(property "Value" "CamButton"
 			(at 176.53 63.4999 0)
 			(effects
@@
 	)
 	(symbol
+		(lib_id "power:GND")
+		(at 154.94 50.8 0)
+		(unit 1)
+		(exclude_from_sim no)
+		(in_bom yes)
+		(on_board yes)
+		(dnp no)
+		(property "Reference" "#PWR011"
+			(at 154.94 57.15 0)
+			(effects
+				(font
+					(size 1.27 1.27)
+				)
+				(hide yes)
+			)
+		)
+		(property "Value" "GND"
+			(at 154.94 55.118 0)
+			(effects
+				(font
+					(size 1.27 1.27)
+				)
+			)
+		)
+		(property "Footprint" ""
+			(at 154.94 50.8 0)
+			(effects
+				(font
+					(size 1.27 1.27)
+				)
+				(hide yes)
+			)
+		)
+		(property "Datasheet" ""
+			(at 154.94 50.8 0)
+			(effects
+				(font
+					(size 1.27 1.27)
+				)
+				(hide yes)
+			)
+		)
+		(property "Description" "Power symbol creates a global label with name \"GND\" , ground"
+			(at 154.94 50.8 0)
+			(effects
+				(font
+					(size 1.27 1.27)
+				)
+				(hide yes)
+			)
+		)
+		(pin "1"
+		)
+		(instances
+			(project "VacuumATM_wCoinDispenser"
+				(path "/175bafae-da8e-452c-ba6d-56d020edb106"
+					(reference "#PWR011")
+					(unit 1)
+				)
+			)
+		)
+	)
+	(symbol
 		(lib_id "power:VBUS")
 		(at 170.18 78.74 90)
@@
 					(unit 1)
 				)
+			)
+		)
+	)
+	(symbol
+		(lib_id "Connector:Screw_Terminal_01x02")
+		(at 165.1 45.72 0)
+		(unit 1)
+		(exclude_from_sim no)
+		(in_bom yes)
+		(on_board yes)
+		(dnp no)
+		(fields_autoplaced yes)
+		(property "Reference" "J6"
+			(at 167.64 45.7199 0)
+			(effects
+				(font
+					(size 1.27 1.27)
+				)
+				(justify left)
+			)
+		)
+		(property "Value" "ResetButton"
+			(at 167.64 48.2599 0)
+			(effects
+				(font
+					(size 1.27 1.27)
+				)
+				(justify left)
+			)
+		)
+		(property "Footprint" "TerminalBlock_Phoenix:TerminalBlock_Phoenix_MKDS-1,5-2_1x02_P5.00mm_Horizontal"
+			(at 165.1 45.72 0)
+			(effects
+				(font
+					(size 1.27 1.27)
+				)
+				(hide yes)
+			)
+		)
+		(property "Datasheet" "~"
+			(at 165.1 45.72 0)
+			(effects
+				(font
+					(size 1.27 1.27)
+				)
+				(hide yes)
+			)
+		)
+		(property "Description" "Generic screw terminal, single row, 01x02, script generated (kicad-library-utils/schlib/autogen/connector/)"
+			(at 165.1 45.72 0)
+			(effects
+				(font
+					(size 1.27 1.27)
+				)
+				(hide yes)
+			)
+		)
+		(pin "2"
+		)
+		(pin "1"
+		)
+		(instances
+			(project "VacuumATM_wCoinDispenser"
+				(path "/175bafae-da8e-452c-ba6d-56d020edb106"
+					(reference "J6")
+					(unit 1)
+				)

Commit message: Redesigned PCB, made Gerber files
Parts:
- J1, J4, J5, J6: footprint TerminalBlock_Phoenix:TerminalBlock_Phoenix_MKDS-1,5-2_1x02_P5.00mm_Horizontal -> TerminalBlock_Phoenix:TerminalBlock_Phoenix_MPT-0,5-2-2.54_1x02_P2.54mm_Horizontal
- J2, J3: footprint TerminalBlock_Phoenix:TerminalBlock_Phoenix_MKDS-1,5-3-5.08_1x03_P5.08mm_Horizontal -> TerminalBlock_Phoenix:TerminalBlock_Phoenix_MPT-0,5-3-2.54_1x03_P2.54mm_Horizontal
Changed lines of the file:
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@@
 			)
 		)
-		(property "Footprint" "TerminalBlock_Phoenix:TerminalBlock_Phoenix_MKDS-1,5-2_1x02_P5.00mm_Horizontal"
+		(property "Footprint" "TerminalBlock_Phoenix:TerminalBlock_Phoenix_MPT-0,5-2-2.54_1x02_P2.54mm_Horizontal"
 			(at 173.99 60.96 0)
 			(effects
@@
 			)
 		)
-		(property "Footprint" "TerminalBlock_Phoenix:TerminalBlock_Phoenix_MKDS-1,5-2_1x02_P5.00mm_Horizontal"
+		(property "Footprint" "TerminalBlock_Phoenix:TerminalBlock_Phoenix_MPT-0,5-2-2.54_1x02_P2.54mm_Horizontal"
 			(at 93.98 52.07 0)
 			(effects
@@
 			)
 		)
-		(property "Footprint" "TerminalBlock_Phoenix:TerminalBlock_Phoenix_MKDS-1,5-3-5.08_1x03_P5.08mm_Horizontal"
+		(property "Footprint" "TerminalBlock_Phoenix:TerminalBlock_Phoenix_MPT-0,5-3-2.54_1x03_P2.54mm_Horizontal"
 			(at 93.98 60.96 0)
 			(effects
@@
 			)
 		)
-		(property "Footprint" "TerminalBlock_Phoenix:TerminalBlock_Phoenix_MKDS-1,5-3-5.08_1x03_P5.08mm_Horizontal"
+		(property "Footprint" "TerminalBlock_Phoenix:TerminalBlock_Phoenix_MPT-0,5-3-2.54_1x03_P2.54mm_Horizontal"
 			(at 175.26 78.74 0)
 			(effects
@@
 			)
 		)
-		(property "Footprint" "TerminalBlock_Phoenix:TerminalBlock_Phoenix_MKDS-1,5-2_1x02_P5.00mm_Horizontal"
+		(property "Footprint" "TerminalBlock_Phoenix:TerminalBlock_Phoenix_MPT-0,5-2-2.54_1x02_P2.54mm_Horizontal"
 			(at 93.98 45.72 0)
 			(effects
@@
 			)
 		)
-		(property "Footprint" "TerminalBlock_Phoenix:TerminalBlock_Phoenix_MKDS-1,5-2_1x02_P5.00mm_Horizontal"
+		(property "Footprint" "TerminalBlock_Phoenix:TerminalBlock_Phoenix_MPT-0,5-2-2.54_1x02_P2.54mm_Horizontal"
 			(at 165.1 45.72 0)
 			(effects

Commit message: Updated KiCAD files
Parts:
- A1: value Adafruit_Feather_Generic -> Photon2; footprint Module:Adafruit_Feather_WithMountingHoles -> Particle:Photon2; symbol MCU_Module:Adafruit_Feather_Generic -> Particle:Photon2
Connections:
- net at J2.1 (Pin_1): now also A1.19 (D2); no longer A1.21 (D2)
- net at J4.1 (Pin_1): now also A1.21 (D4); no longer A1.19 (D0)
Other:
- moved on the sheet: J2, J4
Changed lines of the file:
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@@
 	(wire
 		(pts
-			(xy 99.06 63.5) (xy 100.33 63.5)
-		)
-		(stroke
-			(width 0)
-			(type default)
-		)
-	)
-	(wire
-		(pts
-			(xy 99.06 45.72) (xy 111.76 45.72)
+			(xy 99.06 41.91) (xy 100.33 41.91)
+		)
+		(stroke
+			(width 0)
+			(type default)
+		)
+	)
+	(wire
+		(pts
+			(xy 157.48 60.96) (xy 157.48 73.66)
+		)
+		(stroke
+			(width 0)
+			(type default)
+		)
+	)
+	(wire
+		(pts
+			(xy 170.18 81.28) (xy 146.05 81.28)
+		)
+		(stroke
+			(width 0)
+			(type default)
+		)
+	)
+	(wire
+		(pts
+			(xy 100.33 41.91) (xy 100.33 43.18)
+		)
+		(stroke
+			(width 0)
+			(type default)
+		)
+	)
+	(wire
+		(pts
+			(xy 170.18 71.12) (xy 166.37 71.12)
+		)
+		(stroke
+			(width 0)
+			(type default)
+		)
+	)
+	(wire
+		(pts
+			(xy 110.49 55.88) (xy 120.65 55.88)
+		)
+		(stroke
+			(width 0)
+			(type default)
+		)
+	)
+	(wire
+		(pts
+			(xy 99.06 58.42) (xy 120.65 58.42)
+		)
+		(stroke
+			(width 0)
+			(type default)
+		)
+	)
+	(wire
+		(pts
+			(xy 110.49 52.07) (xy 110.49 55.88)
+		)
+		(stroke
+			(width 0)
+			(type default)
+		)
+	)
+	(wire
+		(pts
+			(xy 160.02 48.26) (xy 154.94 48.26)
+		)
+		(stroke
+			(width 0)
+			(type default)
+		)
+	)
+	(wire
+		(pts
+			(xy 160.02 45.72) (xy 146.05 45.72)
 		)
 		(stroke
@@
 	(wire
 		(pts
-			(xy 157.48 60.96) (xy 157.48 73.66)
-		)
-		(stroke
-			(width 0)
-			(type default)
-		)
-	)
-	(wire
-		(pts
-			(xy 170.18 81.28) (xy 146.05 81.28)
-		)
-		(stroke
-			(width 0)
-			(type default)
-		)
-	)
-	(wire
-		(pts
-			(xy 100.33 63.5) (xy 100.33 64.77)
-		)
-		(stroke
-			(width 0)
-			(type default)
-		)
-	)
-	(wire
-		(pts
-			(xy 170.18 71.12) (xy 166.37 71.12)
-		)
-		(stroke
-			(width 0)
-			(type default)
-		)
-	)
-	(wire
-		(pts
-			(xy 111.76 45.72) (xy 111.76 53.34)
-		)
-		(stroke
-			(width 0)
-			(type default)
-		)
-	)
-	(wire
-		(pts
-			(xy 110.49 55.88) (xy 120.65 55.88)
-		)
-		(stroke
-			(width 0)
-			(type default)
-		)
-	)
-	(wire
-		(pts
-			(xy 110.49 52.07) (xy 110.49 55.88)
-		)
-		(stroke
-			(width 0)
-			(type default)
-		)
-	)
-	(wire
-		(pts
-			(xy 160.02 48.26) (xy 154.94 48.26)
-		)
-		(stroke
-			(width 0)
-			(type default)
-		)
-	)
-	(wire
-		(pts
-			(xy 160.02 45.72) (xy 146.05 45.72)
-		)
-		(stroke
-			(width 0)
-			(type default)
-		)
-	)
-	(wire
-		(pts
-			(xy 99.06 58.42) (xy 120.65 58.42)
+			(xy 99.06 36.83) (xy 111.76 36.83)
+		)
+		(stroke
+			(width 0)
+			(type default)
+		)
+	)
+	(wire
+		(pts
+			(xy 111.76 36.83) (xy 111.76 53.34)
 		)
 		(stroke
@@
 	(symbol
 		(lib_id "Connector:Screw_Terminal_01x03")
-		(at 93.98 60.96 0)
+		(at 93.98 39.37 0)
 		(mirror y)
 		(unit 1)
@@
 		(fields_autoplaced yes)
 		(property "Reference" "J2"
-			(at 91.44 59.6899 0)
+			(at 91.44 38.0999 0)
 			(effects
 				(font
@@
 		)
 		(property "Value" "Neopixel"
-			(at 91.44 62.2299 0)
+			(at 91.44 40.6399 0)
 			(effects
 				(font
@@
 		)
 		(property "Footprint" "TerminalBlock_Phoenix:TerminalBlock_Phoenix_MPT-0,5-3-2.54_1x03_P2.54mm_Horizontal"
-			(at 93.98 60.96 0)
+			(at 93.98 39.37 0)
 			(effects
 				(font
@@
 		)
 		(property "Datasheet" "~"
-			(at 93.98 60.96 0)
+			(at 93.98 39.37 0)
 			(effects
 				(font
@@
 		)
 		(property "Description" "Generic screw terminal, single row, 01x03, script generated (kicad-library-utils/schlib/autogen/connector/)"
-			(at 93.98 60.96 0)
+			(at 93.98 39.37 0)
 			(effects
 				(font
@@
 	(symbol
 		(lib_id "power:GND")
-		(at 100.33 64.77 0)
+		(at 100.33 43.18 0)
 		(mirror y)
 		(unit 1)
@@
 		(dnp no)
 		(property "Reference" "#PWR07"
-			(at 100.33 71.12 0)
+			(at 100.33 49.53 0)
 			(effects
 				(font
@@
 		)
 		(property "Value" "GND"
-			(at 100.33 69.088 0)
+			(at 100.33 47.498 0)
 			(effects
 				(font
@@
 		)
 		(property "Footprint" ""
-			(at 100.33 64.77 0)
+			(at 100.33 43.18 0)
 			(effects
 				(font
@@
 		)
 		(property "Datasheet" ""
-			(at 100.33 64.77 0)
+			(at 100.33 43.18 0)
 			(effects
 				(font
@@
 		)
 		(property "Description" "Power symbol creates a global label with name \"GND\" , ground"
-			(at 100.33 64.77 0)
+			(at 100.33 43.18 0)
 			(effects
 				(font
@@
 	(symbol
 		(lib_id "power:+3.3V")
-		(at 99.06 48.26 270)
+		(at 99.06 60.96 270)
 		(mirror x)
 		(unit 1)
@@
 		(fields_autoplaced yes)
 		(property "Reference" "#PWR09"
-			(at 95.25 48.26 0)
+			(at 95.25 60.96 0)
 			(effects
 				(font
@@
 		)
 		(property "Value" "+3.3V"
-			(at 102.87 48.2599 90)
+			(at 102.87 60.9599 90)
 			(effects
 				(font
@@
 		)
 		(property "Footprint" ""
-			(at 99.06 48.26 0)
+			(at 99.06 60.96 0)
 			(effects
 				(font
@@
 		)
 		(property "Datasheet" ""
-			(at 99.06 48.26 0)
+			(at 99.06 60.96 0)
 			(effects
 				(font
@@
 		)
 		(property "Description" "Power symbol creates a global label with name \"+3.3V\""
-			(at 99.06 48.26 0)
+			(at 99.06 60.96 0)
 			(effects
 				(font
@@
 	(symbol
 		(lib_id "power:VBUS")
-		(at 99.06 60.96 270)
+		(at 99.06 39.37 270)
 		(mirror x)
 		(unit 1)
@@
 		(fields_autoplaced yes)
 		(property "Reference" "#PWR06"
-			(at 95.25 60.96 0)
+			(at 95.25 39.37 0)
 			(effects
 				(font
@@
 		)
 		(property "Value" "VBUS"
-			(at 102.87 60.9599 90)
+			(at 102.87 39.3699 90)
 			(effects
 				(font
@@
 		)
 		(property "Footprint" ""
-			(at 99.06 60.96 0)
+			(at 99.06 39.37 0)
 			(effects
 				(font
@@
 		)
 		(property "Datasheet" ""
-			(at 99.06 60.96 0)
+			(at 99.06 39.37 0)
 			(effects
 				(font
@@
 		)
 		(property "Description" "Power symbol creates a global label with name \"VBUS\""
-			(at 99.06 60.96 0)
+			(at 99.06 39.37 0)
 			(effects
 				(font
@@
 	)
 	(symbol
-		(lib_id "MCU_Module:Adafruit_Feather_Generic")
+		(lib_id "Particle:Photon2")
 		(at 133.35 73.66 0)
 		(unit 1)
@@
 			)
 		)
-		(property "Value" "Adafruit_Feather_Generic"
+		(property "Value" "Photon2"
 			(at 135.5441 109.22 0)
 			(effects
@@
 			)
 		)
-		(property "Footprint" "Module:Adafruit_Feather_WithMountingHoles"
+		(property "Footprint" "Particle:Photon2"
 			(at 135.89 107.95 0)
 			(effects
@@
 			)
 		)
-		(property "Datasheet" "https://cdn-learn.adafruit.com/downloads/pdf/adafruit-feather.pdf"
-			(at 133.35 93.98 0)
+		(property "Datasheet" "https://docs.particle.io/reference/datasheets/wi-fi/photon-2-datasheet/"
+			(at 137.668 114.3 0)
 			(effects
 				(font
@@
 		)
 		(property "Description" "Microcontroller module in various flavor, generic symbol"
-			(at 133.35 73.66 0)
+			(at 134.112 72.898 0)
 			(effects
 				(font
@@
 	(symbol
 		(lib_id "Connector:Screw_Terminal_01x02")
-		(at 93.98 45.72 0)
+		(at 93.98 58.42 0)
 		(mirror y)
 		(unit 1)
@@
 		(fields_autoplaced yes)
 		(property "Reference" "J4"
-			(at 91.44 45.7199 0)
+			(at 91.44 58.4199 0)
 			(effects
 				(font
@@
 		)
 		(property "Value" "User2_Button"
-			(at 91.44 48.2599 0)
+			(at 91.44 60.9599 0)
 			(effects
 				(font
@@
 		)
 		(property "Footprint" "TerminalBlock_Phoenix:TerminalBlock_Phoenix_MPT-0,5-2-2.54_1x02_P2.54mm_Horizontal"
-			(at 93.98 45.72 0)
+			(at 93.98 58.42 0)
 			(effects
 				(font
@@
 		)
 		(property "Datasheet" "~"
-			(at 93.98 45.72 0)
+			(at 93.98 58.42 0)
 			(effects
 				(font
@@
 		)
 		(property "Description" "Generic screw terminal, single row, 01x02, script generated (kicad-library-utils/schlib/autogen/connector/)"
-			(at 93.98 45.72 0)
-			(effects
-				(font
+			(at 93.98 58.42 0)
+			(effects
+				(font
